Commit message: Simulacao refeita para ficar na mesma etapa que estava no projeto anterior

File: src/roboserv_description/urdf/macros.xacro (robot description, xacro)
@@ -1,77 +1,120 @@
 <?xml version="1.0"?>
 <robot>
-<!--Definicoes de inercia-->
-<!--Cilindro-->
-  <macro name="cylinder_inertia" params="m r h">
-    <inertia  ixx="${m*(3*r*r+h*h)/12}" ixy = "0" ixz = "0"
-      iyy="${m*(3*r*r+h*h)/12}" iyz = "0"
-      izz="${m*r*r/2}"
-    />
-  </macro>
-<!--Caixa-->
-  <macro name="box_inertia" params="m x y z">
-    <inertia  ixx="${m*(y*y+z*z)/12}" ixy = "0" ixz = "0"
-      iyy="${m*(x*x+z*z)/12}" iyz = "0"
-      izz="${m*(x*x+z*z)/12}"
-    />
-  </macro>
-<!--Esfera-->
-  <macro name="sphere_inertia" params="m r">
-    <inertia  ixx="${2*m*r*r/5}" ixy = "0" ixz = "0"
-      iyy="${2*m*r*r/5}" iyz = "0"
-      izz="${2*m*r*r/5}"
-    />
-  </macro>
-<!--Dinamicas-->
-<!--Rodas-->
-  <macro name="wheel" params="lr tY">
-    <link name="${lr}_wheel">
-      <collision>
-        <origin xyz="0 0 0" rpy="0 ${PI/2} ${PI/2}" />
-        <geometry>
-          <cylinder length="${wheelWidth}" radius="${wheelRadius}"/>
-        </geometry>
-      </collision>
-      <visual>
-        <origin xyz="0 0 0" rpy="0 ${PI/2} ${PI/2}" />
-        <geometry>
-          <cylinder length="${wheelWidth}" radius="${wheelRadius}"/>
-        </geometry>
-        <material name="black"/>
-      </visual>
-      <inertial>
-        <origin xyz="0 0 0" rpy="0 ${PI/2} ${PI/2}" />
-        <mass value="${wheelMass}"/>
-        <cylinder_inertia m="${wheelMass}" r="${wheelRadius}" h="${wheelWidth}"/>
-      </inertial>
-    </link>
-<!--Define as propriedades do Gazebo-->
-    <gazebo reference="${lr}_wheel">
-      <mu1 value="1.0"/>
-      <mu2 value="1.0"/>
-      <kp  value="10000000.0" />
-      <kd  value="1.0" />
-      <fdir1 value="1 0 0"/>
-      <material>Gazebo/Black</material>
-    </gazebo>
-<!--Dinamica das Juncoes da roda com o chassi-->
-    <joint name="${lr}_wheel_hinge" type="continuous">
-      <parent link="chassis"/>
-      <child link="${lr}_wheel"/>
-    <origin xyz="${-wheelPos+chassisLength/2} ${tY*wheelWidth/2+tY*chassisWidth/2} ${wheelRadius}" rpy="0 0 0" />
-      <axis xyz="0 1 0" rpy="0 0 0" />
-      <limit effort="10000" velocity="10000"/>
-      <joint_properties damping="0.0" friction="0.0"/>
-    </joint>
-    <transmission name="${lr}_trans">
-      <type>transmission_interface/SimpleTransmission</type>
-      <joint name="${lr}_wheel_hinge">
-        <hardwareInterface>EffortJointInterface</hardwareInterface>
-      </joint>
-      <actuator name="${lr}Motor">
-        <hardwareInterface>EffortJointInterface</hardwareInterface>
-        <mechanicalReduction>10</mechanicalReduction>
-      </actuator>
-    </transmission>
-  </macro>
+	<!--Criando um cilindro-->
+	<macro name="create_cylinder" params="name mass radius length px py pz wr wp wy">
+		<collision name="${name}_collision">
+			<origin xyz = "${px} ${py} ${pz}" rpy="${wr} ${wp} ${wy}"/>
+			<geometry>
+				<cylinder radius="${radius}" length="${length}"/>
+			</geometry>
+		</collision>
+		<visual name="${name}_visual">
+			<origin xyz = "${px} ${py} ${pz}" rpy="${wr} ${wp} ${wy}"/>
+			<geometry>
+				<cylinder radius="${radius}" length="${length}"/>
+			</geometry>
+		</visual>
+		<inertial>
+			<origin xyz = "${px} ${py} ${pz}" rpy="${wr} ${wp} ${wy}"/>
+			<mass value="${mass}"/>
+			<inertia
+				ixx="${mass*(3*radius*radius+length*length)/12}" ixy = "0" ixz = "0"
+				iyy="${mass*(3*radius*radius+length*length)/12}" iyz = "0"
+				izz="${mass*radius*radius/2}" />
+		</inertial>
+	</macro>
+	<!--Criando uma caixa-->
+	<macro name="create_box" params="name mass size_x size_y size_z px py pz wr wp wy">
+		<collision name="${name}_collision">
+			<origin xyz = "${px} ${py} ${pz}" rpy="${wr} ${wp} ${wy}"/>
+			<geometry>
+				<box size="${size_x} ${size_y} ${size_z}"/>
+			</geometry>
+		</collision>
+		<visual name="${name}_visual">
+			<origin xyz = "${px} ${py} ${pz}" rpy="${wr} ${wp} ${wy}"/>
+			<geometry>
+				<box size="${size_x} ${size_y} ${size_z}"/>
+			</geometry>
+		</visual>
+		<inertial>
+			<origin xyz = "${px} ${py} ${pz+0.1}" rpy="${wr} ${wp} ${wy}"/>
+			<mass value="${mass}"/>
+			<inertia
+				ixx="${mass*(size_y*size_y+size_z*size_z)/12}" ixy = "0" ixz = "0"
+				iyy="${mass*(size_x*size_x+size_z*size_z)/12}" iyz = "0"
+				izz="${mass*(size_x*size_x+size_z*size_z)/12}" />
+		</inertial>
+	</macro>
+	<!--Criando uma esfera-->
+	<macro name="create_sphere" params="name mass radius px py pz wr wp wy">
+		<collision name="${name}_collision">
+			<origin xyz = "${px} ${py} ${pz}" rpy="${wr} ${wp} ${wy}"/>
+			<geometry>
+				<sphere radius="${radius}"/>
+			</geometry>
+			<surface>
+				<friction>
+					<ode>
+						<mu>0</mu>
+						<mu2>0</mu2>
+						<slip1>1.0</slip1>
+						<slip2>1.0</slip2>
+					</ode>
+				</friction>
+			</surface>
+		</collision>
+		<visual name="${name}_visual">
+			<origin xyz = "${px} ${py} ${pz}" rpy="${wr} ${wp} ${wy}"/>
+			<geometry>
+				<sphere radius="${radius}"/>
+			</geometry>
+		</visual>
+		<inertial>
+			<origin xyz = "${px} ${py} ${pz}" rpy="${wr} ${wp} ${wy}"/>
+			<mass value="${mass}"/>
+			<inertia
+				ixx="${mass*radius*radius*2/5}" ixy = "0" ixz = "0"
+				iyy="${mass*radius*radius*2/5}" iyz = "0"
+				izz="${mass*radius*radius*2/5}" />
+		</inertial>
+	</macro>
+	<!--Criando uma roda-->
+	<macro name="create_wheel" params="name mass radius length body_name body_size_x body_size_y wheel_pos_x wheel_side whell_spacing">
+		<!--Cria um cilindro-->
+		<link name="${name}">
+			<create_cylinder name="${name}" mass="${mass}" radius="${radius}" length="${length}"
+						  px="0" py="0" pz="0" wr="0" wp="${pi/2}" wy="${pi/2}"/>
+		</link>
+		<!--Cria uma referencia no Gazebo-->
+		<gazebo reference="${name}">
+			<mu1 value="1.0"/>
+			<mu2 value="1.0"/>
+			<kp  value="1000000.0" />
+			<kd  value="100.0" />
+			<max_vel value="1.0" />
+			<fdir1 value="0 0 0"/>
+			<material>Gazebo/Black</material>
+		</gazebo>
+		<!--Cria a juncao com o corpo-->
+		<joint name="${name}_hinge" type="continuous">
+			<parent link="${body_name}"/>
+			<child link="${name}"/>
+			<origin xyz="${-wheel_pos_x+body_size_x/2} ${(length/2+body_size_y/2+whell_spacing)*wheel_side} 0" rpy="0 0 0" />
+			<axis xyz="0 1 0" rpy="0 0 0" />
+			<limit effort="10000" velocity="10000"/>
+			<joint_properties damping="1.0" friction="1.0"/>
+		</joint>
+		<!--Cria uma configuracao de transmissao-->
+		<transmission name="${name}_trans">
+			<type>transmission_interface/SimpleTransmission</type>
+			<joint name="${name}_hinge">
+				<hardwareInterface>EffortJointInterface</hardwareInterface>
+			</joint>
+			<actuator name="${name}_motor">
+				<hardwareInterface>EffortJointInterface</hardwareInterface>
+				<mechanicalReduction>10</mechanicalReduction>
+			</actuator>
+		</transmission>
+	</macro>
 </robot>

File: src/roboserv_description/urdf/roboserv.xacro (robot description, xacro)
@@ -1,189 +1,97 @@
 <?xml version='1.0'?>
 <robot name="roboserv" xmlns:xacro="http://www.ros.org/wiki/xacro">
-<!--Incluir os outros arquivos necessarios-->
-  <xacro:include filename="$(find roboserv_description)/urdf/roboserv.gazebo" />
-  <xacro:include filename="$(find roboserv_description)/urdf/materials.xacro" />
-  <xacro:include filename="$(find roboserv_description)/urdf/macros.xacro" />
-<!-- ESTRUTURA DO ROBO -->
-<!--Chassi-->
-  <link name='chassis'>
-    <pose>0 0 0.1 0 0 0</pose>
-    <inertial>
-      <mass value="10.0"/>
-      <origin xyz="0.0 0 0.1" rpy=" 0 0 0"/>
-      <inertia
-          ixx="0.5" ixy="0" ixz="0"
-          iyy="1.0" iyz="0"
-          izz="0.1"
-      />
-    </inertial>
-    <collision name='collision'>
-      <geometry>
-        <box size=".4 .2 .1"/>
-      </geometry>
-    </collision>
-    <visual name='chassis_visual'>
-      <origin xyz="0 0 0" rpy=" 0 0 0"/>
-      <geometry>
-        <box size=".4 .2 .1"/>
-      </geometry>
-    </visual>
-<!--Roda esferica frontal-->
-    <collision name='caster_collision'>
-      <origin xyz="-0.15 0 -0.05" rpy=" 0 0 0"/>
-      <geometry>
-        <sphere radius="0.05"/>
-      </geometry>
-      <surface>
-        <friction>
-          <ode>
-            <mu>0</mu>
-            <mu2>0</mu2>
-            <slip1>1.0</slip1>
-            <slip2>1.0</slip2>
-          </ode>
-        </friction>
-      </surface>
-    </collision>
-    <visual name='caster_visual'>
-      <origin xyz="-0.15 0 -0.05" rpy=" 0 0 0"/>
-      <geometry>
-        <sphere radius="0.05"/>
-      </geometry>
-    </visual>
-  </link>
-<!--Roda esquerda-->
-  <link name="left_wheel">
-    <!--origin xyz="0.1 0.13 0.1" rpy="0 1.5707 1.5707"/-->
-    <collision name="collision">
-      <origin xyz="0 0 0" rpy="0 1.5707 1.5707"/>
-      <geometry>
-        <cylinder radius="0.1" length="0.05"/>
-      </geometry>
-    </collision>
-    <visual name="left_wheel_visual">
-      <origin xyz="0 0 0" rpy="0 1.5707 1.5707"/>
-      <geometry>
-        <cylinder radius="0.1" length="0.05"/>
-      </geometry>
-    </visual>
-    <inertial>
-      <origin xyz="0 0 0" rpy="0 1.5707 1.5707"/>
-      <mass value="5"/>
-      <cylinder_inertia m="5" r="0.1" h="0.05"/>
-      <inertia
-        ixx="1.0" ixy="0.0" ixz="0.0"
-        iyy="1.0" iyz="0.0"
-        izz="1.0"/>
-    </inertial>
-  </link>
-<!--Roda direita-->
-  <link name="right_wheel">
-    <!--origin xyz="0.1 -0.13 0.1" rpy="0 1.5707 1.5707"/-->
-    <collision name="collision">
-      <origin xyz="0 0 0" rpy="0 1.5707 1.5707"/>
-      <geometry>
-        <cylinder radius="0.1" length="0.05"/>
-      </geometry>
-    </collision>
-    <visual name="right_wheel_visual">
-      <origin xyz="0 0 0" rpy="0 1.5707 1.5707"/>
-      <geometry>
-        <cylinder radius="0.1" length="0.05"/>
-      </geometry>
-    </visual>
-    <inertial>
-      <origin xyz="0 0 0" rpy="0 1.5707 1.5707"/>
-      <mass value="5"/>
-      <cylinder_inertia m="5" r="0.1" h="0.05"/>
-      <inertia
-        ixx="1.0" ixy="0.0" ixz="0.0"
-        iyy="1.0" iyz="0.0"
-        izz="1.0"/>
-    </inertial>
-  </link>
-<!-- JUNCOES -->
-<!--Roda esquerda : Chassi-->
-  <joint type="continuous" name="left_wheel_hinge">
-    <origin xyz="0.1 0.15 0" rpy="0 0 0"/>
-    <child link="left_wheel"/>
-    <parent link="chassis"/>
-    <axis xyz="0 1 0" rpy="0 0 0"/>
-    <limit effort="100" velocity="100"/>
-    <joint_properties damping="0.0" friction="0.0"/>
-  </joint>
-<!--Roda direita : Chassi-->
-  <joint type="continuous" name="right_wheel_hinge">
-    <origin xyz="0.1 -0.15 0" rpy="0 0 0"/>
-    <child link="right_wheel"/>
-    <parent link="chassis"/>
-    <axis xyz="0 1 0" rpy="0 0 0"/>
-    <limit effort="100" velocity="100"/>
-    <joint_properties damping="0.0" friction="0.0"/>
-  </joint>
-<!-- PLUGINS -->
-<!--Kinect-->
-  <xacro:property name="kinect_cam_py" value="-0.0125"/>
-  <!-- Parameterised in part by the values in turtlebot_properties.urdf.xacro -->
+	<!--Incluir os outros arquivos necessarios-->
+	<xacro:include filename="$(find roboserv_description)/urdf/roboserv.gazebo" />
+	<xacro:include filename="$(find roboserv_description)/urdf/materials.xacro" />
+	<xacro:include filename="$(find roboserv_description)/urdf/macros.xacro" />
+	<xacro:property name="robot_name" value="robo_link" />
+	<xacro:property name="body_size_x" value="0.4" />
+	<xacro:property name="body_size_y" value="0.2" />
+	<xacro:property name="body_size_z" value="0.1" />
+	<xacro:property name="body_mass" value="5.0" />
+	<xacro:property name="caster_radius" value="0.05" />
+	<xacro:property name="caster_mass" value="1.0" />
+	<xacro:property name="wheel_radius" value="0.1" />
+	<xacro:property name="wheel_length" value="0.05" />
+	<xacro:property name="wheel_mass" value="5.0" />
+	<!--Corpo do robo-->
+	<link name="${robot_name}">
+		<!--Posicao inicial do carro-->
+    	<pose>0 0 0.1 0 0 0</pose>
+		<!--Chassi-->
+		<xacro:create_box name="chassis" mass="${body_mass}" size_x="${body_size_x}" size_y="${body_size_y}" size_z="${body_size_z}"
+						  px="0" py="0" pz="0" wr="0" wp="0" wy="0"/>
+		<!--Roda esferica frontal-->
+		<xacro:create_sphere name="caster" mass="${caster_mass}" radius="${caster_radius}"
+						  px="-0.15" py="0" pz="-0.05" wr="0" wp="0" wy="0"/>
+	</link>
+	<!--Roda esquerda-->
+	<xacro:create_wheel name="left_wheel" mass="${wheel_mass}" radius="${wheel_radius}" length="${wheel_length}"
+						body_name="${robot_name}" body_size_x="${body_size_x}" body_size_y="${body_size_y}"
+						wheel_pos_x="0.015" wheel_side = "1" whell_spacing="0.02"/>
+	<!--Roda direita-->
+	<xacro:create_wheel name="right_wheel" mass="${wheel_mass}" radius="${wheel_radius}" length="${wheel_length}"
+						body_name="${robot_name}" body_size_x="${body_size_x}" body_size_y="${body_size_y}"
+						wheel_pos_x="0.015" wheel_side = "-1" whell_spacing="0.02"/>
+	<!--Kinect-->
+	<!--Declarando as propriedades-->
+	<xacro:property name="kinect_cam_py" value="-0.0125"/>
 	<xacro:property name="cam_px" value="0.18" />
-    <xacro:property name="cam_py" value="-0.0125" />
+	<xacro:property name="cam_py" value="-0.0125" />
 	<xacro:property name="cam_pz" value="0.0870" />
 	<xacro:property name="cam_or" value="0" />
 	<xacro:property name="cam_op" value="0" />
 	<xacro:property name="cam_oy" value="0" />
-    <joint name="camera_rgb_joint" type="fixed">
-      <origin xyz="${cam_px} ${cam_py} ${cam_pz}" rpy="${cam_or} ${cam_op} ${cam_oy}"/>
-      <parent link="chassis"/>
-      <child link="camera_rgb_frame" />
-    </joint>
-    <link name="camera_rgb_frame"/>
-    <joint name="camera_rgb_optical_joint" type="fixed">
-      <origin xyz="0 0 0" rpy="${-pi/2} 0 ${-pi/2}" />
-      <parent link="camera_rgb_frame" />
-      <child link="camera_rgb_optical_frame" />
-    </joint>
-    <link name="camera_rgb_optical_frame"/>
-    <joint name="camera_joint" type="fixed">
-      <origin xyz="-0.031 ${-kinect_cam_py} -0.016" rpy="0 0 0"/>
-      <parent link="camera_rgb_frame"/>
-      <child link="camera_link"/>
-    </joint>
-      <link name="camera_link">
-      <visual>
-       <origin xyz="0 0 0" rpy="0 0 ${pi/2}"/>
-        <geometry>
-         <mesh filename="package://turtlebot_description/meshes/sensors/kinect.dae"/>
-        </geometry>
-      </visual>
-  	  <collision>
-        <origin xyz="0.0 0.0 0.0" rpy="0 0 0"/>
-  	    <geometry>
-  	      <box size="0.07271 0.27794 0.073"/>
-  	    </geometry>
-  	  </collision>
-      <inertial>
-        <mass value="0.564" />
-        <origin xyz="0 0 0" />
-        <inertia ixx="0.003881243" ixy="0.0" ixz="0.0"
-                 iyy="0.000498940" iyz="0.0"
-                 izz="0.003879257" />
-      </inertial>
-    </link>
-    <!-- The fixed joints & links below are usually published by static_transformers launched by the OpenNi launch
-         files. However, for Gazebo simulation we need them, so we add them here.
-         (Hence, don't publish them additionally!) -->
+	<!--Criando as juncoes-->
+	<!--Chassi -> Camera RGB-->
+	<joint name="camera_rgb_joint" type="fixed">
+		<origin xyz="${cam_px} ${cam_py} ${cam_pz}" rpy="${cam_or} ${cam_op} ${cam_oy}"/>
+		<parent link="${robot_name}"/>
+		<child link="camera_rgb_frame" />
+	</joint>
+	<!--Camera RGB -> Camera link (corpo do Kinect)-->
+	<joint name="camera_joint" type="fixed">
+		<origin xyz="-0.031 ${-kinect_cam_py} -0.016" rpy="0 0 0"/>
+		<parent link="camera_rgb_frame"/>
+		<child link="camera_link"/>
+	</joint>
+	<!--Camera RGB -> Camera RGB optica-->
+	<joint name="camera_rgb_optical_joint" type="fixed">
+		<origin xyz="0 0 0" rpy="${-pi/2} 0 ${-pi/2}" />
+		<parent link="camera_rgb_frame" />
+		<child link="camera_rgb_optical_frame" />
+	</joint>
+	<!--Camera RGB -> Camera de profundidade-->
 	<joint name="camera_depth_joint" type="fixed">
-	  <origin xyz="0 ${2 * -kinect_cam_py} 0" rpy="0 0 0" />
-	  <parent link="camera_rgb_frame" />
-	  <child link="camera_depth_frame" />
+		<origin xyz="0 ${2 * -kinect_cam_py} 0" rpy="0 0 0" />
+		<parent link="camera_rgb_frame" />
+		<child link="camera_depth_frame" />
 	</joint>
+	<!--Camera de profundidade -> Camera de profundidade optica-->
+	<joint name="camera_depth_optical_joint" type="fixed">
+		<origin xyz="0 0 0" rpy="${-pi/2} 0 ${-pi/2}" />
+		<parent link="camera_depth_frame" />
+		<child link="camera_depth_optical_frame" />
+	</joint>
+	<!--Criando os frames-->
+	<link name="camera_rgb_frame"/>
+	<link name="camera_rgb_optical_frame"/>
 	<link name="camera_depth_frame"/>
-	<joint name="camera_depth_optical_joint" type="fixed">
-	  <origin xyz="0 0 0" rpy="${-pi/2} 0 ${-pi/2}" />
-	  <parent link="camera_depth_frame" />
-	  <child link="camera_depth_optical_frame" />
-	</joint>
 	<link name="camera_depth_optical_frame"/>
-	<!-- Kinect sensor for simulation -->
+	<!--Criando o corpo do Kinect-->
+	<link name="camera_link">
+		<visual>
+			<origin xyz="0 0 0" rpy="0 0 ${pi/2}"/>
+			<geometry>
+				<mesh filename="package://turtlebot_description/meshes/sensors/kinect.dae"/>
+			</geometry>
+		</visual>
+		<collision>
+			<origin xyz="0.0 0.0 0.0" rpy="0 0 0"/>
+			<geometry>
+				<box size="0.07271 0.27794 0.073"/>
+			</geometry>
+		</collision>
+	</link>
 	<turtlebot_sim_3dsensor/>
 </robot>
