Commit message: Path planning funcional - v1, robo alterado

File: src/roboserv_description/urdf/macros.xacro (robot description, xacro)
@@ -81,5 +81,5 @@
 	</macro>
 	<!--Criando uma roda-->
-	<macro name="create_wheel" params="name mass radius length body_name body_size_x body_size_y wheel_pos_x wheel_side whell_spacing">
+	<macro name="create_wheel" params="name mass radius length body_name body_size_y wheel_pos_z wheel_pos_x wheel_side whell_spacing">
 		<!--Cria um cilindro-->
 		<link name="${name}">
@@ -101,5 +101,5 @@
 			<parent link="${body_name}"/>
 			<child link="${name}"/>
-			<origin xyz="${-wheel_pos_x+body_size_x/2} ${(length/2+body_size_y/2+whell_spacing)*wheel_side} 0" rpy="0 0 0" />
+			<origin xyz="0 ${(length/2+body_size_y/2+whell_spacing)*wheel_side} ${wheel_pos_z}" rpy="0 0 0" />
 			<axis xyz="0 1 0" rpy="0 0 0" />
 			<limit effort="10000" velocity="10000"/>
@@ -118,3 +118,31 @@
 		</transmission>
 	</macro>
+	<!--Criando um sensor de distancia-->
+	<macro name="create_ir" params="name body_name lenght height ang_degree">
+		<joint name="${name}" type="fixed">
+			<axis xyz="0 1 0" />
+			<origin rpy="0 0 ${ang_degree*pi/180}" xyz="${lenght*cos(ang_degree*pi/180)} ${lenght*sin(ang_degree*pi/180)} ${height}" />
+			<parent link="${body_name}"/>
+			<child link="${name}"/>
+		</joint>
+		<link name="${name}">
+			<visual>
+				<origin xyz="0 0 0" rpy="0 0 0"/>
+				<geometry>
+					<box size="0.01 0.01 0.01"/>
+				</geometry>
+			</visual>
+			<collision>
+				<origin xyz="0 0 0" rpy="0 0 0"/>
+				<geometry>
+					<box size="0.01 0.01 0.01"/>
+				</geometry>
+			</collision>
+			<inertial>
+				<mass value="1e-5" />
+				<origin xyz="0 0 0" rpy="0 0 0"/>
+				<inertia ixx="1e-6" ixy="0" ixz="0" iyy="1e-6" iyz="0" izz="1e-6" />
+			</inertial>
+		</link>
+	</macro>
 </robot>

File: src/roboserv_description/urdf/roboserv.xacro (robot description, xacro)
@@ -6,31 +6,34 @@
 	<xacro:include filename="$(find roboserv_description)/urdf/macros.xacro" />
 	<xacro:property name="robot_name" value="robo_link" />
-	<xacro:property name="body_size_x" value="0.4" />
-	<xacro:property name="body_size_y" value="0.2" />
-	<xacro:property name="body_size_z" value="0.1" />
+	<xacro:property name="body_radius" value="0.2" />
+	<xacro:property name="body_length" value="0.1" />
 	<xacro:property name="body_mass" value="5.0" />
-	<xacro:property name="caster_radius" value="0.05" />
+	<xacro:property name="caster_radius" value="0.03" />
+	<xacro:property name="caster_z" value="-0.03" />
 	<xacro:property name="caster_mass" value="1.0" />
-	<xacro:property name="wheel_radius" value="0.1" />
-	<xacro:property name="wheel_length" value="0.05" />
-	<xacro:property name="wheel_mass" value="5.0" />
+	<xacro:property name="wheel_radius" value="0.05" />
+	<xacro:property name="wheel_z" value="-0.0105" />
+	<xacro:property name="wheel_length" value="0.02" />
+	<xacro:property name="wheel_mass" value="4.0" />
 	<!--Corpo do robo-->
 	<link name="${robot_name}">
 		<!--Posicao inicial do carro-->
     	<pose>0 0 0.1 0 0 0</pose>
-		<!--Chassi-->
-		<xacro:create_box name="chassis" mass="${body_mass}" size_x="${body_size_x}" size_y="${body_size_y}" size_z="${body_size_z}"
+		<xacro:create_cylinder name="chassis" mass="${body_mass}" radius="${body_radius}" length="${body_length}"
 						  px="0" py="0" pz="0" wr="0" wp="0" wy="0"/>
 		<!--Roda esferica frontal-->
 		<xacro:create_sphere name="caster" mass="${caster_mass}" radius="${caster_radius}"
-						  px="-0.15" py="0" pz="-0.05" wr="0" wp="0" wy="0"/>
+						  px="-0.15" py="0" pz="${caster_z}" wr="0" wp="0" wy="0"/>
+		<!--Roda esferica traseira-->
+		<xacro:create_sphere name="caster" mass="${caster_mass}" radius="${caster_radius}"
+						  px="0.15" py="0" pz="${caster_z}" wr="0" wp="0" wy="0"/>
 	</link>
 	<!--Roda esquerda-->
 	<xacro:create_wheel name="left_wheel" mass="${wheel_mass}" radius="${wheel_radius}" length="${wheel_length}"
-						body_name="${robot_name}" body_size_x="${body_size_x}" body_size_y="${body_size_y}"
+						body_name="${robot_name}" body_size_y="${body_radius}" wheel_pos_z="${wheel_z}"
 						wheel_pos_x="0.015" wheel_side = "1" whell_spacing="0.02"/>
 	<!--Roda direita-->
 	<xacro:create_wheel name="right_wheel" mass="${wheel_mass}" radius="${wheel_radius}" length="${wheel_length}"
-						body_name="${robot_name}" body_size_x="${body_size_x}" body_size_y="${body_size_y}"
+						body_name="${robot_name}" body_size_y="${body_radius}" wheel_pos_z="${wheel_z}"
 						wheel_pos_x="0.015" wheel_side = "-1" whell_spacing="0.02"/>
 	<!--Kinect-->
@@ -95,3 +98,56 @@
 	</link>
 	<turtlebot_sim_3dsensor/>
+	<!--Sensor Infravermelho-->
+	<xacro:create_ir name="distSensor_R"  body_name="${robot_name}" lenght="${body_radius}" height="${body_length/2}" ang_degree="-45"/>
+	<xacro:create_ir name="distSensor_FR" body_name="${robot_name}" lenght="${body_radius}" height="${body_length/2}" ang_degree="-25"/>
+	<xacro:create_ir name="distSensor_F"  body_name="${robot_name}" lenght="${body_radius}" height="${body_length/2}" ang_degree="0"/>
+	<xacro:create_ir name="distSensor_FL" body_name="${robot_name}" lenght="${body_radius}" height="${body_length/2}" ang_degree="25"/>
+	<xacro:create_ir name="distSensor_L"  body_name="${robot_name}" lenght="${body_radius}" height="${body_length/2}" ang_degree="45"/>
+	<!--joint name="ir_front_joint" type="fixed">
+		<axis xyz="0 1 0" />
+		<origin rpy="0 0 ${pi/4}" xyz="${body_radius} 0 ${body_length/2}" />
+		<parent link="robo_link"/>
+		<child link="base_ir_front"/>
+	</joint>
+	<link name="base_ir_front">
+		<collision>
+		  <origin xyz="0 0 0" rpy="0 0 0"/>
+		  <geometry>
+			<box size="0.01 0.01 0.01"/>
+		  </geometry>
+		</collision>    <visual>
+		  <origin xyz="0 0 0" rpy="0 0 0"/>
+		  <geometry>
+			<box size="0.01 0.01 0.01"/>
+		  </geometry>
+		</visual>    <inertial>
+		  <mass value="1e-5" />
+		  <origin xyz="0 0 0" rpy="0 0 0"/>
+		  <inertia ixx="1e-6" ixy="0" ixz="0" iyy="1e-6" iyz="0"      izz="1e-6" />
+		</inertial>
+	</link-->
+	<!--Sensor Sonar
+	<joint name="sonar_front_joint" type="fixed">
+		<axis xyz="0 1 0" />
+		<origin rpy="0 0 0" xyz="${body_radius} 0 ${body_length/2}" />
+		<parent link="robo_link"/>
+		<child link="base_sonar_front"/>
+	</joint>
+	<link name="base_sonar_front">
+		<collision>
+		  <origin xyz="0 0 0" rpy="0 0 0"/>
+		  <geometry>
+			<box size="0.01 0.01 0.01"/>
+		  </geometry>
+		</collision>    <visual>
+		  <origin xyz="0 0 0" rpy="0 0 0"/>
+		  <geometry>
+			<box size="0.01 0.01 0.01"/>
+		  </geometry>
+		</visual>    <inertial>
+		  <mass value="1e-5" />
+		  <origin xyz="0 0 0" rpy="0 0 0"/>
+		  <inertia ixx="1e-6" ixy="0" ixz="0" iyy="1e-6" iyz="0" izz="1e-6" />
+		</inertial>
+	 </link>-->
 </robot>

Commit message: Protoipo funcionando com path planning e rampa de aceleracao

File: src/roboserv_description/urdf/macros.xacro (robot description, xacro)
@@ -87,14 +87,4 @@
 						  px="0" py="0" pz="0" wr="0" wp="${pi/2}" wy="${pi/2}"/>
 		</link>
-		<!--Cria uma referencia no Gazebo-->
-		<gazebo reference="${name}">
-			<mu1 value="1.0"/>
-			<mu2 value="1.0"/>
-			<kp  value="1000000.0" />
-			<kd  value="100.0" />
-			<max_vel value="1.0" />
-			<fdir1 value="0 0 0"/>
-			<material>Gazebo/Black</material>
-		</gazebo>
 		<!--Cria a juncao com o corpo-->
 		<joint name="${name}_hinge" type="continuous">

File: src/roboserv_description/urdf/roboserv.xacro (robot description, xacro)
@@ -2,11 +2,13 @@
 <robot name="roboserv" xmlns:xacro="http://www.ros.org/wiki/xacro">
 	<!-- Argumentos -->
-	<xacro:arg name="use_sim_camera" default="true" />
-	<xacro:arg name="use_sim_distSensors" default="true" />
+	<xacro:arg name="using_simulation" default="1"/>
+	<xacro:property name="using_simulation" value="$(arg using_simulation)" />
 	<!--Incluir os outros arquivos necessarios-->
-	<xacro:include filename="$(find roboserv_description)/urdf/roboserv.gazebo" /> <!-- use_sim_camera:=$(arg use_sim_camera) use_sim_distSensors:=$(arg use_sim_distSensors)" /-->
+	<xacro:if value="${using_simulation==1}">
+		<xacro:include filename="$(find roboserv_description)/urdf/roboserv.gazebo" />
+	</xacro:if>
 	<xacro:include filename="$(find roboserv_description)/urdf/materials.xacro" />
 	<xacro:include filename="$(find roboserv_description)/urdf/macros.xacro" />
-	<xacro:property name="robot_name" value="robo_link" />
+	<xacro:property name="robot_name" value="base_link" />
 	<xacro:property name="body_radius" value="0.2"/>
 	<xacro:property name="body_length" value="0.1" />
@@ -40,14 +42,61 @@
 						body_name="${robot_name}" body_size_y="${body_radius}" wheel_pos_z="${wheel_z}"
 						wheel_pos_x="0.015" wheel_side = "-1" whell_spacing="0.02"/>
-	<xacro:if value="$(arg use_sim_camera)">
+	<!--Propriedades da câmera-->
+	<xacro:property name="cam_px" value="0.18" />
+	<xacro:property name="cam_py" value="-0.0125" />
+	<xacro:property name="cam_pz" value="0.7" />
+	<xacro:property name="cam_or" value="0" />
+	<xacro:property name="cam_op" value="0" />
+	<xacro:property name="cam_oy" value="0" />
+	<xacro:if value="${using_simulation==0}">
+		<!--ZED-->
+		<!-- Camera Center -->
+		<joint name="zed_camera_center_joint" type="fixed">
+			<parent link="base_link"/>
+			<child link="zed_camera_center"/>
+			<origin xyz="${cam_px} ${cam_py} ${cam_pz}" rpy="${cam_or} ${cam_op} ${cam_oy}"/>
+		</joint>
+		<link name="zed_camera_center">
+			<visual>
+				<origin xyz="0 0 0" rpy="0 0 0"/>
+				<geometry>
+					<mesh filename="package://zed_wrapper/urdf/models/ZED.stl" />
+				</geometry>
+				<material name="light_grey">
+					<color rgba="0.8 0.8 0.8 0.8"/>
+				</material>
+			</visual>
+		</link>
+		<!-- Left Camera -->
+		<joint name="zed_left_camera_joint" type="fixed">
+			<parent link="zed_camera_center"/>
+			<child link="zed_left_camera_frame"/>
+			<origin xyz="0 0.06 0" rpy="0 0 0" />
+		</joint>
+		<link name="zed_left_camera_frame" />
+			<joint name="zed_left_camera_optical_joint" type="fixed">
+				<origin xyz="0 0 0" rpy="-1.57079632679 0.0 -1.57079632679"/>
+				<parent link="zed_left_camera_frame"/>
+				<child link="zed_left_camera_optical_frame"/>
+			</joint>
+		<link name="zed_left_camera_optical_frame"/>
+		<!-- Right Camera -->
+		<joint name="zed_right_camera_joint" type="fixed">
+			<parent link="zed_camera_center"/>
+			<child link="zed_right_camera_frame"/>
+			<origin xyz="0 -0.06 0" rpy="0 0 0" />
+		</joint>
+		<link name="zed_right_camera_frame" />
+			<joint name="zed_right_camera_optical_joint" type="fixed">
+				<origin xyz="0 0 0" rpy="-1.57079632679 0.0 -1.57079632679"/>
+				<parent link="zed_right_camera_frame"/>
+				<child link="zed_right_camera_optical_frame"/>
+			</joint>
+		<link name="zed_right_camera_optical_frame"/>
+	</xacro:if>
+	<xacro:if value="${using_simulation==1}">
 		<!--Kinect-->
 		<!--Declarando as propriedades-->
 		<xacro:property name="kinect_cam_py" value="-0.0125"/>
-		<xacro:property name="cam_px" value="0.18" />
-		<xacro:property name="cam_py" value="-0.0125" />
-		<xacro:property name="cam_pz" value="0.0870" />
-		<xacro:property name="cam_or" value="0" />
-		<xacro:property name="cam_op" value="0" />
-		<xacro:property name="cam_oy" value="0" />
 		<!--Criando as juncoes-->
 		<!--Chassi -> Camera RGB-->
@@ -109,50 +158,3 @@
 	<xacro:create_ir name="distSensor_FL" body_name="${robot_name}" lenght="${body_radius}" height="${body_length/2}" ang_degree="25"/>
 	<xacro:create_ir name="distSensor_L"  body_name="${robot_name}" lenght="${body_radius}" height="${body_length/2}" ang_degree="45"/>
-	<!--joint name="ir_front_joint" type="fixed">
-		<axis xyz="0 1 0" />
-		<origin rpy="0 0 ${pi/4}" xyz="${body_radius} 0 ${body_length/2}" />
-		<parent link="robo_link"/>
-		<child link="base_ir_front"/>
-	</joint>
-	<link name="base_ir_front">
-		<collision>
-		  <origin xyz="0 0 0" rpy="0 0 0"/>
-		  <geometry>
-			<box size="0.01 0.01 0.01"/>
-		  </geometry>
-		</collision>    <visual>
-		  <origin xyz="0 0 0" rpy="0 0 0"/>
-		  <geometry>
-			<box size="0.01 0.01 0.01"/>
-		  </geometry>
-		</visual>    <inertial>
-		  <mass value="1e-5" />
-		  <origin xyz="0 0 0" rpy="0 0 0"/>
-		  <inertia ixx="1e-6" ixy="0" ixz="0" iyy="1e-6" iyz="0"      izz="1e-6" />
-		</inertial>
-	</link-->
-	<!--Sensor Sonar
-	<joint name="sonar_front_joint" type="fixed">
-		<axis xyz="0 1 0" />
-		<origin rpy="0 0 0" xyz="${body_radius} 0 ${body_length/2}" />
-		<parent link="robo_link"/>
-		<child link="base_sonar_front"/>
-	</joint>
-	<link name="base_sonar_front">
-		<collision>
-		  <origin xyz="0 0 0" rpy="0 0 0"/>
-		  <geometry>
-			<box size="0.01 0.01 0.01"/>
-		  </geometry>
-		</collision>    <visual>
-		  <origin xyz="0 0 0" rpy="0 0 0"/>
-		  <geometry>
-			<box size="0.01 0.01 0.01"/>
-		  </geometry>
-		</visual>    <inertial>
-		  <mass value="1e-5" />
-		  <origin xyz="0 0 0" rpy="0 0 0"/>
-		  <inertia ixx="1e-6" ixy="0" ixz="0" iyy="1e-6" iyz="0" izz="1e-6" />
-		</inertial>
-	 </link>-->
 </robot>
