Commit message: Criando o modelo real do robo no urdf

File: src/roboserv_description/urdf/macros.xacro (robot description, xacro)
@@ -1,24 +1,50 @@
 <?xml version="1.0"?>
-<robot>
+<robot xmlns:xacro="http://www.ros.org/wiki/xacro">
 	<!--Criando um cilindro-->
-	<macro name="create_cylinder" params="name mass radius length px py pz wr wp wy">
+	<macro name="create_cylinder" params="name radius height pos_x pos_y pos_z wr wp wy density">
+		<xacro:property name="mass" value="${radius*radius*pi*height*density}"/>
 		<collision name="${name}_collision">
-			<origin xyz = "${px} ${py} ${pz}" rpy="${wr} ${wp} ${wy}"/>
+			<origin xyz = "${pos_x} ${pos_y} ${pos_z}" rpy="${wr} ${wp} ${wy}"/>
 			<geometry>
-				<cylinder radius="${radius}" length="${length}"/>
+				<cylinder radius="${radius}" length="${height}"/>
 			</geometry>
 		</collision>
 		<visual name="${name}_visual">
-			<origin xyz = "${px} ${py} ${pz}" rpy="${wr} ${wp} ${wy}"/>
+			<origin xyz = "${pos_x} ${pos_y} ${pos_z}" rpy="${wr} ${wp} ${wy}"/>
 			<geometry>
-				<cylinder radius="${radius}" length="${length}"/>
+				<cylinder radius="${radius}" length="${height}"/>
 			</geometry>
 		</visual>
 		<inertial>
-			<origin xyz = "${px} ${py} ${pz}" rpy="${wr} ${wp} ${wy}"/>
+			<origin xyz = "${pos_x} ${pos_y} ${pos_z}" rpy="${wr} ${wp} ${wy}"/>
 			<mass value="${mass}"/>
 			<inertia
-				ixx="${mass*(3*radius*radius+length*length)/12}" ixy = "0" ixz = "0"
-				iyy="${mass*(3*radius*radius+length*length)/12}" iyz = "0"
+				ixx="${mass*(3*radius*radius+height*height)/12}" ixy = "0" ixz = "0"
+				iyy="${mass*(3*radius*radius+height*height)/12}" iyz = "0"
+				izz="${mass*radius*radius/2}" />
+		</inertial>
+	</macro>
+	<!--Criando uma peça-->
+	<macro name="create_mesh" params="name size_x size_y size_z dist_x dist_y dist_z wr wp wy density">
+		<xacro:property name="radius" value="${(size_x+size_y)/4}"/>
+		<xacro:property name="mass" value="${radius*radius*pi*size_z*density*0.6}"/>
+		<collision name="${name}_collision">
+			<origin xyz = "${dist_x-size_x/2} ${dist_y-size_y/2} ${dist_z-size_z}" rpy="${wr} ${wp} ${wy}"/>
+			<geometry>
+				<cylinder radius="${radius}" length="${size_z}"/>
+			</geometry>
+		</collision>
+		<visual name="${name}_visual">
+			<origin xyz = "${dist_x-size_x} ${-dist_y+size_y} ${dist_z-size_z}" rpy="${wr-pi/2} ${wp} ${wy-pi/2}"/>
+			<geometry>
+				<mesh filename="package://roboserv_description/urdf/models/dae/${name}.dae" scale="0.001 0.001 0.001"/>
+			</geometry>
+		</visual>
+		<inertial>
+			<origin xyz = "${dist_x-size_x/2} ${dist_y-size_y/2} ${dist_z-size_z}" rpy="${wr} ${wp} ${wy}"/>
+			<mass value="${mass}"/>
+			<inertia
+				ixx="${mass*(3*radius*radius+size_z*size_z)/12}" ixy = "0" ixz = "0"
+				iyy="${mass*(3*radius*radius+size_z*size_z)/12}" iyz = "0"
 				izz="${mass*radius*radius/2}" />
 		</inertial>
@@ -46,4 +72,7 @@
 				izz="${mass*(size_x*size_x+size_z*size_z)/12}" />
 		</inertial>
+		<material name="black">
+			<color rgba="0 0 0 0"/>
+		</material>
 	</macro>
 	<!--Criando uma esfera-->
@@ -84,6 +113,5 @@
 		<!--Cria um cilindro-->
 		<link name="${name}">
-			<create_cylinder name="${name}" mass="${mass}" radius="${radius}" length="${length}"
-						  px="0" py="0" pz="0" wr="0" wp="${pi/2}" wy="${pi/2}"/>
+			<create_cylinder name="${name}" radius="${radius}" height="${length}" pos_x="0" pos_y="0" pos_z="0" wr="0" wp="${pi/2}" wy="${pi/2}" density="600"/>
 		</link>
 		<!--Cria a juncao com o corpo-->

File: src/roboserv_description/urdf/roboserv_old.xacro (robot description, xacro)
@@ -25,44 +25,18 @@
 		<!--Posicao inicial do carro-->
     	<pose>0 0 0.5 0 0 0</pose>
-		<xacro:create_mesh name="BaseLV1" size_x="0.5" size_y="0.3988" size_z="0.01" dist_x="0.2" dist_y="0.1994" dist_z="-0.02905" wr="0" wp="0" wy="0" density="650" />
-<xacro:create_mesh name="BaseLV2" size_x="0.5" size_y="0.3988" size_z="0.01" dist_x="0.2" dist_y="0.1994" dist_z="0.01905" wr="0" wp="0" wy="0" density="650" />
-<xacro:create_mesh name="BaseLV3" size_x="0.435" size_y="0.4" size_z="0.00635" dist_x="0.135" dist_y="0.2" dist_z="0.25505" wr="0" wp="0" wy="0" density="650" />
-<xacro:create_mesh name="BaseLV4" size_x="0.25" size_y="0.25" size_z="0.00635" dist_x="0.0008" dist_y="0.125" dist_z="0.7114" wr="0" wp="0" wy="0" density="650" />
-<xacro:create_mesh name="Suporte" size_x="0.12607" size_y="0.12607" size_z="0.009" dist_x="-0.06117" dist_y="0.063035" dist_z="0.20605" wr="0" wp="0" wy="0" density="650" />
-<xacro:create_mesh name="PlatMovelLV1" size_x="0.2054" size_y="0.19661" size_z="0.01" dist_x="-0.0215" dist_y="0.098305" dist_z="0.33745" wr="0" wp="0" wy="0" density="650" />
-<xacro:create_mesh name="PlatMovelLV2" size_x="0.25" size_y="0.25" size_z="0.01" dist_x="0.0008" dist_y="0.125" dist_z="0.76745" wr="0" wp="0" wy="0" density="650" />
-<xacro:create_cylinder name="C_LV1_1" radius="0.00635" height="0.0381" pos_x="0.14" pos_y="0.05443" pos_z="-0.02" wr="0" wp="0" wy="0" density="800" />
-<xacro:create_cylinder name="C_LV1_2" radius="0.00635" height="0.0381" pos_x="0.14" pos_y="-0.05443" pos_z="-0.02" wr="0" wp="0" wy="0" density="800" />
-<xacro:create_cylinder name="C_LV1_3" radius="0.00635" height="0.0381" pos_x="0.05" pos_y="0.1142" pos_z="-0.02" wr="0" wp="0" wy="0" density="800" />
-<xacro:create_cylinder name="C_LV1_4" radius="0.00635" height="0.0381" pos_x="0.05" pos_y="-0.1142" pos_z="-0.02" wr="0" wp="0" wy="0" density="800" />
-<xacro:create_cylinder name="C_LV1_5" radius="0.00635" height="0.0381" pos_x="-0.07" pos_y="0.1142" pos_z="-0.02" wr="0" wp="0" wy="0" density="800" />
-<xacro:create_cylinder name="C_LV1_6" radius="0.00635" height="0.0381" pos_x="-0.07" pos_y="-0.1142" pos_z="-0.02" wr="0" wp="0" wy="0" density="800" />
-<xacro:create_cylinder name="C_LV1_7" radius="0.00635" height="0.0381" pos_x="-0.19" pos_y="0.07843" pos_z="-0.02" wr="0" wp="0" wy="0" density="800" />
-<xacro:create_cylinder name="C_LV1_8" radius="0.00635" height="0.0381" pos_x="-0.19" pos_y="-0.07843" pos_z="-0.02" wr="0" wp="0" wy="0" density="800" />
-<xacro:create_cylinder name="C_LV1_9" radius="0.00635" height="0.0381" pos_x="-0.27" pos_y="0" pos_z="-0.02" wr="0" wp="0" wy="0" density="800" />
-<xacro:create_cylinder name="C_LV2_1" radius="0.00635" height="0.226" pos_x="0.085" pos_y="0.115" pos_z="0.12205" wr="0" wp="0" wy="0" density="800" />
-<xacro:create_cylinder name="C_LV2_2" radius="0.00635" height="0.226" pos_x="0.085" pos_y="-0.115" pos_z="0.12205" wr="0" wp="0" wy="0" density="800" />
-<xacro:create_cylinder name="C_LV2_3" radius="0.00635" height="0.226" pos_x="-0.125" pos_y="0.115" pos_z="0.12205" wr="0" wp="0" wy="0" density="800" />
-<xacro:create_cylinder name="C_LV2_4" radius="0.00635" height="0.226" pos_x="-0.125" pos_y="-0.115" pos_z="0.12205" wr="0" wp="0" wy="0" density="800" />
-<xacro:create_cylinder name="C_LV2_5" radius="0.00635" height="0.226" pos_x="-0.2492" pos_y="0" pos_z="0.12205" wr="0" wp="0" wy="0" density="800" />
-<xacro:create_cylinder name="C_SPT_1" radius="0.00635" height="0.05" pos_x="-0.07117" pos_y="0" pos_z="0.22005" wr="0" wp="0" wy="0" density="800" />
-<xacro:create_cylinder name="C_SPT_2" radius="0.00635" height="0.05" pos_x="-0.125" pos_y="0.05303" pos_z="0.22005" wr="0" wp="0" wy="0" density="800" />
-<xacro:create_cylinder name="C_SPT_3" radius="0.00635" height="0.05" pos_x="-0.125" pos_y="-0.05303" pos_z="0.22005" wr="0" wp="0" wy="0" density="800" />
-<xacro:create_cylinder name="C_SPT_4" radius="0.00635" height="0.05" pos_x="-0.17723" pos_y="0" pos_z="0.22005" wr="0" wp="0" wy="0" density="800" />
-<xacro:create_cylinder name="C_LV3_1" radius="0.00635" height="0.448" pos_x="-0.05349" pos_y="0.07071" pos_z="0.4754" wr="0" wp="0" wy="0" density="800" />
-<xacro:create_cylinder name="C_LV3_2" radius="0.00635" height="0.448" pos_x="-0.05349" pos_y="-0.07071" pos_z="0.4754" wr="0" wp="0" wy="0" density="800" />
-<xacro:create_cylinder name="C_LV3_3" radius="0.00635" height="0.448" pos_x="-0.19491" pos_y="0.07071" pos_z="0.4754" wr="0" wp="0" wy="0" density="800" />
-<xacro:create_cylinder name="C_LV3_4" radius="0.00635" height="0.448" pos_x="-0.19491" pos_y="-0.07071" pos_z="0.4754" wr="0" wp="0" wy="0" density="800" />
-<xacro:create_cylinder name="C_GUIA_1" radius="0.00635" height="0.5" pos_x="-0.04635" pos_y="0" pos_z="0.5014" wr="0" wp="0" wy="0" density="800" />
-<xacro:create_cylinder name="C_GUIA_2" radius="0.00635" height="0.5" pos_x="-0.20135" pos_y="0" pos_z="0.5014" wr="0" wp="0" wy="0" density="800" />
-<xacro:create_cylinder name="C_PLT_1" radius="0.00635" height="0.42" pos_x="-0.06632" pos_y="0.02252" pos_z="0.54745" wr="0" wp="0" wy="0" density="800" />
-<xacro:create_cylinder name="C_PLT_2" radius="0.00635" height="0.42" pos_x="-0.1242" pos_y="0.0804" pos_z="0.54745" wr="0" wp="0" wy="0" density="800" />
-<xacro:create_cylinder name="C_PLT_3" radius="0.00635" height="0.42" pos_x="-0.1242" pos_y="0.0804" pos_z="0.54745" wr="0" wp="0" wy="0" density="800" />
-<xacro:create_cylinder name="C_PLT_4" radius="0.00635" height="0.42" pos_x="-0.18208" pos_y="-0.02252" pos_z="0.54745" wr="0" wp="0" wy="0" density="800" />
-<xacro:create_cylinder name="C_BODY" radius="0.0125" height="0.506" pos_x="-0.1242" pos_y="0" pos_z="0.49055" wr="0" wp="0" wy="0" density="800" />
-		<!--
+		<xacro:create_mesh name="BaseLV1" mass="${body_mass}" radius="${body_radius}" length="${body_length}"
+						  px="-0.3" py="0.2" pz="0.06" wr="${-pi/2}" wp="0" wy="${-pi/2}"/>
+		<xacro:create_mesh name="BaseLV2" mass="${body_mass}" radius="${body_radius}" length="${body_length}"
+						  px="-0.3" py="0.2" pz="0.1" wr="${-pi/2}" wp="0" wy="${-pi/2}"/>
+		<xacro:create_mesh name="BaseLV3" mass="${body_mass}" radius="${body_radius}" length="${body_length}"
+						  px="-0.3" py="0.2" pz="0.2" wr="${-pi/2}" wp="0" wy="${-pi/2}"/>
+		<xacro:create_mesh name="PlatMovelLV1" mass="${body_mass}" radius="${body_radius}" length="${body_length}"
+						  px="-0.3" py="0.2" pz="0.3" wr="${-pi/2}" wp="0" wy="${-pi/2}"/>
+		<xacro:create_mesh name="PlatMovelLV2" mass="${body_mass}" radius="${body_radius}" length="${body_length}"
+						  px="-0.3" py="0.2" pz="0.4" wr="${-pi/2}" wp="0" wy="${-pi/2}"/>
+		<xacro:create_mesh name="SuporteMotorPasso" mass="${body_mass}" radius="${body_radius}" length="${body_length}"
+						  px="-0.3" py="0.2" pz="0.5" wr="${-pi/2}" wp="0" wy="${-pi/2}"/>
 		<xacro:create_cylinder name="chassis" mass="${body_mass}" radius="${body_radius}" length="${body_length}"
 						  px="0" py="0" pz="0" wr="0" wp="0" wy="0"/>
-		-->
 		<!--Roda esferica frontal-->
 		<xacro:create_sphere name="caster" mass="${caster_mass}" radius="${caster_radius}"
