Commit message: Adicionado comunicacao com sensores arduino

File: src/roboserv_description/urdf/roboserv.xacro (robot description, xacro)
@@ -1,10 +1,13 @@
 <?xml version='1.0'?>
 <robot name="roboserv" xmlns:xacro="http://www.ros.org/wiki/xacro">
+	<!-- Argumentos -->
+	<xacro:arg name="use_sim_camera" default="true" />
+	<xacro:arg name="use_sim_distSensors" default="true" />
 	<!--Incluir os outros arquivos necessarios-->
-	<xacro:include filename="$(find roboserv_description)/urdf/roboserv.gazebo" />
+	<xacro:include filename="$(find roboserv_description)/urdf/roboserv.gazebo" /> <!-- use_sim_camera:=$(arg use_sim_camera) use_sim_distSensors:=$(arg use_sim_distSensors)" /-->
 	<xacro:include filename="$(find roboserv_description)/urdf/materials.xacro" />
 	<xacro:include filename="$(find roboserv_description)/urdf/macros.xacro" />
 	<xacro:property name="robot_name" value="robo_link" />
-	<xacro:property name="body_radius" value="0.2" />
+	<xacro:property name="body_radius" value="0.2"/>
 	<xacro:property name="body_length" value="0.1" />
 	<xacro:property name="body_mass" value="5.0" />
@@ -37,65 +40,67 @@
 						body_name="${robot_name}" body_size_y="${body_radius}" wheel_pos_z="${wheel_z}"
 						wheel_pos_x="0.015" wheel_side = "-1" whell_spacing="0.02"/>
-	<!--Kinect-->
-	<!--Declarando as propriedades-->
-	<xacro:property name="kinect_cam_py" value="-0.0125"/>
-	<xacro:property name="cam_px" value="0.18" />
-	<xacro:property name="cam_py" value="-0.0125" />
-	<xacro:property name="cam_pz" value="0.0870" />
-	<xacro:property name="cam_or" value="0" />
-	<xacro:property name="cam_op" value="0" />
-	<xacro:property name="cam_oy" value="0" />
-	<!--Criando as juncoes-->
-	<!--Chassi -> Camera RGB-->
-	<joint name="camera_rgb_joint" type="fixed">
-		<origin xyz="${cam_px} ${cam_py} ${cam_pz}" rpy="${cam_or} ${cam_op} ${cam_oy}"/>
-		<parent link="${robot_name}"/>
-		<child link="camera_rgb_frame" />
-	</joint>
-	<!--Camera RGB -> Camera link (corpo do Kinect)-->
-	<joint name="camera_joint" type="fixed">
-		<origin xyz="-0.031 ${-kinect_cam_py} -0.016" rpy="0 0 0"/>
-		<parent link="camera_rgb_frame"/>
-		<child link="camera_link"/>
-	</joint>
-	<!--Camera RGB -> Camera RGB optica-->
-	<joint name="camera_rgb_optical_joint" type="fixed">
-		<origin xyz="0 0 0" rpy="${-pi/2} 0 ${-pi/2}" />
-		<parent link="camera_rgb_frame" />
-		<child link="camera_rgb_optical_frame" />
-	</joint>
-	<!--Camera RGB -> Camera de profundidade-->
-	<joint name="camera_depth_joint" type="fixed">
-		<origin xyz="0 ${2 * -kinect_cam_py} 0" rpy="0 0 0" />
-		<parent link="camera_rgb_frame" />
-		<child link="camera_depth_frame" />
-	</joint>
-	<!--Camera de profundidade -> Camera de profundidade optica-->
-	<joint name="camera_depth_optical_joint" type="fixed">
-		<origin xyz="0 0 0" rpy="${-pi/2} 0 ${-pi/2}" />
-		<parent link="camera_depth_frame" />
-		<child link="camera_depth_optical_frame" />
-	</joint>
-	<!--Criando os frames-->
-	<link name="camera_rgb_frame"/>
-	<link name="camera_rgb_optical_frame"/>
-	<link name="camera_depth_frame"/>
-	<link name="camera_depth_optical_frame"/>
-	<!--Criando o corpo do Kinect-->
-	<link name="camera_link">
-		<visual>
-			<origin xyz="0 0 0" rpy="0 0 ${pi/2}"/>
-			<geometry>
-				<mesh filename="package://turtlebot_description/meshes/sensors/kinect.dae"/>
-			</geometry>
-		</visual>
-		<collision>
-			<origin xyz="0.0 0.0 0.0" rpy="0 0 0"/>
-			<geometry>
-				<box size="0.07271 0.27794 0.073"/>
-			</geometry>
-		</collision>
-	</link>
-	<turtlebot_sim_3dsensor/>
+	<xacro:if value="$(arg use_sim_camera)">
+		<!--Kinect-->
+		<!--Declarando as propriedades-->
+		<xacro:property name="kinect_cam_py" value="-0.0125"/>
+		<xacro:property name="cam_px" value="0.18" />
+		<xacro:property name="cam_py" value="-0.0125" />
+		<xacro:property name="cam_pz" value="0.0870" />
+		<xacro:property name="cam_or" value="0" />
+		<xacro:property name="cam_op" value="0" />
+		<xacro:property name="cam_oy" value="0" />
+		<!--Criando as juncoes-->
+		<!--Chassi -> Camera RGB-->
+		<joint name="camera_rgb_joint" type="fixed">
+			<origin xyz="${cam_px} ${cam_py} ${cam_pz}" rpy="${cam_or} ${cam_op} ${cam_oy}"/>
+			<parent link="${robot_name}"/>
+			<child link="camera_rgb_frame" />
+		</joint>
+		<!--Camera RGB -> Camera link (corpo do Kinect)-->
+		<joint name="camera_joint" type="fixed">
+			<origin xyz="-0.031 ${-kinect_cam_py} -0.016" rpy="0 0 0"/>
+			<parent link="camera_rgb_frame"/>
+			<child link="camera_link"/>
+		</joint>
+		<!--Camera RGB -> Camera RGB optica-->
+		<joint name="camera_rgb_optical_joint" type="fixed">
+			<origin xyz="0 0 0" rpy="${-pi/2} 0 ${-pi/2}" />
+			<parent link="camera_rgb_frame" />
+			<child link="camera_rgb_optical_frame" />
+		</joint>
+		<!--Camera RGB -> Camera de profundidade-->
+		<joint name="camera_depth_joint" type="fixed">
+			<origin xyz="0 ${2 * -kinect_cam_py} 0" rpy="0 0 0" />
+			<parent link="camera_rgb_frame" />
+			<child link="camera_depth_frame" />
+		</joint>
+		<!--Camera de profundidade -> Camera de profundidade optica-->
+		<joint name="camera_depth_optical_joint" type="fixed">
+			<origin xyz="0 0 0" rpy="${-pi/2} 0 ${-pi/2}" />
+			<parent link="camera_depth_frame" />
+			<child link="camera_depth_optical_frame" />
+		</joint>
+		<!--Criando os frames-->
+		<link name="camera_rgb_frame"/>
+		<link name="camera_rgb_optical_frame"/>
+		<link name="camera_depth_frame"/>
+		<link name="camera_depth_optical_frame"/>
+		<!--Criando o corpo do Kinect-->
+		<link name="camera_link">
+			<visual>
+				<origin xyz="0 0 0" rpy="0 0 ${pi/2}"/>
+				<geometry>
+					<mesh filename="package://turtlebot_description/meshes/sensors/kinect.dae"/>
+				</geometry>
+			</visual>
+			<collision>
+				<origin xyz="0.0 0.0 0.0" rpy="0 0 0"/>
+				<geometry>
+					<box size="0.07271 0.27794 0.073"/>
+				</geometry>
+			</collision>
+		</link>
+		<turtlebot_sim_3dsensor/>
+	</xacro:if>
 	<!--Sensor Infravermelho-->
 	<xacro:create_ir name="distSensor_R"  body_name="${robot_name}" lenght="${body_radius}" height="${body_length/2}" ang_degree="-45"/>

Commit message: + progresso - prototipo andando

File: src/roboserv_description/urdf/roboserv.xacro (robot description, xacro)
@@ -25,4 +25,20 @@
 		<!--Posicao inicial do carro-->
     	<pose>0 0 0.5 0 0 0</pose>
+		<joint name="base_LV1" type="fixed">
+			<parent link="base_link"/>
+			<child link="base_LV1"/>
+			<origin xyz="0 0 0.3" rpy="0 0 0"/>
+		</joint>
+		<link name="base_LV1">
+			<visual>
+				<origin xyz="0 0 0" rpy="0 0 0"/>
+				<geometry>
+					<mesh filename="package://roboserv_description/urdf/models/BaseLV1.stl" />
+				</geometry>
+				<material name="black">
+					<color rgba="0.0 0.0 0.0 0.0"/>
+				</material>
+			</visual>
+		</link>
 		<xacro:create_cylinder name="chassis" mass="${body_mass}" radius="${body_radius}" length="${body_length}"
 						  px="0" py="0" pz="0" wr="0" wp="0" wy="0"/>
@@ -34,16 +50,18 @@
 						  px="0.15" py="0" pz="${caster_z}" wr="0" wp="0" wy="0"/>
 	</link>
-	<!--Roda esquerda-->
-	<xacro:create_wheel name="left_wheel" mass="${wheel_mass}" radius="${wheel_radius}" length="${wheel_length}"
-						body_name="${robot_name}" body_size_y="${body_radius}" wheel_pos_z="${wheel_z}"
-						wheel_pos_x="0.015" wheel_side = "1" whell_spacing="0.02"/>
-	<!--Roda direita-->
-	<xacro:create_wheel name="right_wheel" mass="${wheel_mass}" radius="${wheel_radius}" length="${wheel_length}"
-						body_name="${robot_name}" body_size_y="${body_radius}" wheel_pos_z="${wheel_z}"
-						wheel_pos_x="0.015" wheel_side = "-1" whell_spacing="0.02"/>
+	<xacro:if value="${using_simulation==1}">
+		<!--Roda esquerda-->
+		<xacro:create_wheel name="left_wheel" mass="${wheel_mass}" radius="${wheel_radius}" length="${wheel_length}"
+							body_name="${robot_name}" body_size_y="${body_radius}" wheel_pos_z="${wheel_z}"
+							wheel_pos_x="0.015" wheel_side = "1" whell_spacing="0.02"/>
+		<!--Roda direita-->
+		<xacro:create_wheel name="right_wheel" mass="${wheel_mass}" radius="${wheel_radius}" length="${wheel_length}"
+							body_name="${robot_name}" body_size_y="${body_radius}" wheel_pos_z="${wheel_z}"
+							wheel_pos_x="0.015" wheel_side = "-1" whell_spacing="0.02"/>
+	</xacro:if>
 	<!--Propriedades da câmera-->
-	<xacro:property name="cam_px" value="0.18" />
-	<xacro:property name="cam_py" value="-0.0125" />
-	<xacro:property name="cam_pz" value="0.7" />
+	<xacro:property name="cam_px" value="0" />
+	<xacro:property name="cam_py" value="0" />
+	<xacro:property name="cam_pz" value="0.8" />
 	<xacro:property name="cam_or" value="0" />
 	<xacro:property name="cam_op" value="0" />
@@ -61,5 +79,5 @@
 				<origin xyz="0 0 0" rpy="0 0 0"/>
 				<geometry>
-					<mesh filename="package://zed_wrapper/urdf/models/ZED.stl" />
+					<mesh filename="package://roboserv_description/urdf/models/BaseLV1.stl" />
 				</geometry>
 				<material name="light_grey">
@@ -140,5 +158,5 @@
 				<origin xyz="0 0 0" rpy="0 0 ${pi/2}"/>
 				<geometry>
-					<mesh filename="package://turtlebot_description/meshes/sensors/kinect.dae"/>
+					<mesh filename="package://roboserv_description/urdf/models/BaseLV1.stl"/>
 				</geometry>
 			</visual>
@@ -154,7 +172,5 @@
 	<!--Sensor Infravermelho-->
 	<xacro:create_ir name="distSensor_R"  body_name="${robot_name}" lenght="${body_radius}" height="${body_length/2}" ang_degree="-45"/>
-	<xacro:create_ir name="distSensor_FR" body_name="${robot_name}" lenght="${body_radius}" height="${body_length/2}" ang_degree="-25"/>
 	<xacro:create_ir name="distSensor_F"  body_name="${robot_name}" lenght="${body_radius}" height="${body_length/2}" ang_degree="0"/>
-	<xacro:create_ir name="distSensor_FL" body_name="${robot_name}" lenght="${body_radius}" height="${body_length/2}" ang_degree="25"/>
 	<xacro:create_ir name="distSensor_L"  body_name="${robot_name}" lenght="${body_radius}" height="${body_length/2}" ang_degree="45"/>
 </robot>

Commit message: Corrigindo robo

File: src/roboserv_description/urdf/roboserv.xacro (robot description, xacro)
@@ -25,20 +25,4 @@
 		<!--Posicao inicial do carro-->
     	<pose>0 0 0.5 0 0 0</pose>
-		<joint name="base_LV1" type="fixed">
-			<parent link="base_link"/>
-			<child link="base_LV1"/>
-			<origin xyz="0 0 0.3" rpy="0 0 0"/>
-		</joint>
-		<link name="base_LV1">
-			<visual>
-				<origin xyz="0 0 0" rpy="0 0 0"/>
-				<geometry>
-					<mesh filename="package://roboserv_description/urdf/models/BaseLV1.stl" />
-				</geometry>
-				<material name="black">
-					<color rgba="0.0 0.0 0.0 0.0"/>
-				</material>
-			</visual>
-		</link>
 		<xacro:create_cylinder name="chassis" mass="${body_mass}" radius="${body_radius}" length="${body_length}"
 						  px="0" py="0" pz="0" wr="0" wp="0" wy="0"/>
@@ -79,5 +63,5 @@
 				<origin xyz="0 0 0" rpy="0 0 0"/>
 				<geometry>
-					<mesh filename="package://roboserv_description/urdf/models/BaseLV1.stl" />
+					<mesh filename="package://zed_wrapper/urdf/models/ZED.stl" />
 				</geometry>
 				<material name="light_grey">
@@ -158,5 +142,5 @@
 				<origin xyz="0 0 0" rpy="0 0 ${pi/2}"/>
 				<geometry>
-					<mesh filename="package://roboserv_description/urdf/models/BaseLV1.stl"/>
+					<mesh filename="package://turtlebot_description/meshes/sensors/kinect.dae"/>
 				</geometry>
 			</visual>

Commit message: move_base (algoritmo do path planning) funcionando

File: src/roboserv_description/urdf/roboserv.xacro (robot description, xacro)
@@ -26,39 +26,39 @@
     	<pose>0 0 0.5 0 0 0</pose>
 		<xacro:create_mesh name="BaseLV1" size_x="0.5" size_y="0.3988" size_z="0.01" dist_x="0.2" dist_y="0.1994" dist_z="-0.02905" wr="0" wp="0" wy="0" density="650" />
-<xacro:create_mesh name="BaseLV2" size_x="0.5" size_y="0.3988" size_z="0.01" dist_x="0.2" dist_y="0.1994" dist_z="0.01905" wr="0" wp="0" wy="0" density="650" />
-<xacro:create_mesh name="BaseLV3" size_x="0.435" size_y="0.4" size_z="0.00635" dist_x="0.135" dist_y="0.2" dist_z="0.25505" wr="0" wp="0" wy="0" density="650" />
-<xacro:create_mesh name="BaseLV4" size_x="0.25" size_y="0.25" size_z="0.00635" dist_x="0.0008" dist_y="0.125" dist_z="0.7114" wr="0" wp="0" wy="0" density="650" />
-<xacro:create_mesh name="Suporte" size_x="0.12607" size_y="0.12607" size_z="0.009" dist_x="-0.06117" dist_y="0.063035" dist_z="0.20605" wr="0" wp="0" wy="0" density="650" />
-<xacro:create_mesh name="PlatMovelLV1" size_x="0.2054" size_y="0.19661" size_z="0.01" dist_x="-0.0215" dist_y="0.098305" dist_z="0.33745" wr="0" wp="0" wy="0" density="650" />
-<xacro:create_mesh name="PlatMovelLV2" size_x="0.25" size_y="0.25" size_z="0.01" dist_x="0.0008" dist_y="0.125" dist_z="0.76745" wr="0" wp="0" wy="0" density="650" />
-<xacro:create_cylinder name="C_LV1_1" radius="0.00635" height="0.0381" pos_x="0.14" pos_y="0.05443" pos_z="-0.02" wr="0" wp="0" wy="0" density="800" />
-<xacro:create_cylinder name="C_LV1_2" radius="0.00635" height="0.0381" pos_x="0.14" pos_y="-0.05443" pos_z="-0.02" wr="0" wp="0" wy="0" density="800" />
-<xacro:create_cylinder name="C_LV1_3" radius="0.00635" height="0.0381" pos_x="0.05" pos_y="0.1142" pos_z="-0.02" wr="0" wp="0" wy="0" density="800" />
-<xacro:create_cylinder name="C_LV1_4" radius="0.00635" height="0.0381" pos_x="0.05" pos_y="-0.1142" pos_z="-0.02" wr="0" wp="0" wy="0" density="800" />
-<xacro:create_cylinder name="C_LV1_5" radius="0.00635" height="0.0381" pos_x="-0.07" pos_y="0.1142" pos_z="-0.02" wr="0" wp="0" wy="0" density="800" />
-<xacro:create_cylinder name="C_LV1_6" radius="0.00635" height="0.0381" pos_x="-0.07" pos_y="-0.1142" pos_z="-0.02" wr="0" wp="0" wy="0" density="800" />
-<xacro:create_cylinder name="C_LV1_7" radius="0.00635" height="0.0381" pos_x="-0.19" pos_y="0.07843" pos_z="-0.02" wr="0" wp="0" wy="0" density="800" />
-<xacro:create_cylinder name="C_LV1_8" radius="0.00635" height="0.0381" pos_x="-0.19" pos_y="-0.07843" pos_z="-0.02" wr="0" wp="0" wy="0" density="800" />
-<xacro:create_cylinder name="C_LV1_9" radius="0.00635" height="0.0381" pos_x="-0.27" pos_y="0" pos_z="-0.02" wr="0" wp="0" wy="0" density="800" />
-<xacro:create_cylinder name="C_LV2_1" radius="0.00635" height="0.226" pos_x="0.085" pos_y="0.115" pos_z="0.12205" wr="0" wp="0" wy="0" density="800" />
-<xacro:create_cylinder name="C_LV2_2" radius="0.00635" height="0.226" pos_x="0.085" pos_y="-0.115" pos_z="0.12205" wr="0" wp="0" wy="0" density="800" />
-<xacro:create_cylinder name="C_LV2_3" radius="0.00635" height="0.226" pos_x="-0.125" pos_y="0.115" pos_z="0.12205" wr="0" wp="0" wy="0" density="800" />
-<xacro:create_cylinder name="C_LV2_4" radius="0.00635" height="0.226" pos_x="-0.125" pos_y="-0.115" pos_z="0.12205" wr="0" wp="0" wy="0" density="800" />
-<xacro:create_cylinder name="C_LV2_5" radius="0.00635" height="0.226" pos_x="-0.2492" pos_y="0" pos_z="0.12205" wr="0" wp="0" wy="0" density="800" />
-<xacro:create_cylinder name="C_SPT_1" radius="0.00635" height="0.05" pos_x="-0.07117" pos_y="0" pos_z="0.22005" wr="0" wp="0" wy="0" density="800" />
-<xacro:create_cylinder name="C_SPT_2" radius="0.00635" height="0.05" pos_x="-0.125" pos_y="0.05303" pos_z="0.22005" wr="0" wp="0" wy="0" density="800" />
-<xacro:create_cylinder name="C_SPT_3" radius="0.00635" height="0.05" pos_x="-0.125" pos_y="-0.05303" pos_z="0.22005" wr="0" wp="0" wy="0" density="800" />
-<xacro:create_cylinder name="C_SPT_4" radius="0.00635" height="0.05" pos_x="-0.17723" pos_y="0" pos_z="0.22005" wr="0" wp="0" wy="0" density="800" />
-<xacro:create_cylinder name="C_LV3_1" radius="0.00635" height="0.448" pos_x="-0.05349" pos_y="0.07071" pos_z="0.4754" wr="0" wp="0" wy="0" density="800" />
-<xacro:create_cylinder name="C_LV3_2" radius="0.00635" height="0.448" pos_x="-0.05349" pos_y="-0.07071" pos_z="0.4754" wr="0" wp="0" wy="0" density="800" />
-<xacro:create_cylinder name="C_LV3_3" radius="0.00635" height="0.448" pos_x="-0.19491" pos_y="0.07071" pos_z="0.4754" wr="0" wp="0" wy="0" density="800" />
-<xacro:create_cylinder name="C_LV3_4" radius="0.00635" height="0.448" pos_x="-0.19491" pos_y="-0.07071" pos_z="0.4754" wr="0" wp="0" wy="0" density="800" />
-<xacro:create_cylinder name="C_GUIA_1" radius="0.00635" height="0.5" pos_x="-0.04635" pos_y="0" pos_z="0.5014" wr="0" wp="0" wy="0" density="800" />
-<xacro:create_cylinder name="C_GUIA_2" radius="0.00635" height="0.5" pos_x="-0.20135" pos_y="0" pos_z="0.5014" wr="0" wp="0" wy="0" density="800" />
-<xacro:create_cylinder name="C_PLT_1" radius="0.00635" height="0.42" pos_x="-0.06632" pos_y="0.02252" pos_z="0.54745" wr="0" wp="0" wy="0" density="800" />
-<xacro:create_cylinder name="C_PLT_2" radius="0.00635" height="0.42" pos_x="-0.1242" pos_y="0.0804" pos_z="0.54745" wr="0" wp="0" wy="0" density="800" />
-<xacro:create_cylinder name="C_PLT_3" radius="0.00635" height="0.42" pos_x="-0.1242" pos_y="0.0804" pos_z="0.54745" wr="0" wp="0" wy="0" density="800" />
-<xacro:create_cylinder name="C_PLT_4" radius="0.00635" height="0.42" pos_x="-0.18208" pos_y="-0.02252" pos_z="0.54745" wr="0" wp="0" wy="0" density="800" />
-<xacro:create_cylinder name="C_BODY" radius="0.0125" height="0.506" pos_x="-0.1242" pos_y="0" pos_z="0.49055" wr="0" wp="0" wy="0" density="800" />
+		<xacro:create_mesh name="BaseLV2" size_x="0.5" size_y="0.3988" size_z="0.01" dist_x="0.2" dist_y="0.1994" dist_z="0.01905" wr="0" wp="0" wy="0" density="650" />
+		<xacro:create_mesh name="BaseLV3" size_x="0.435" size_y="0.4" size_z="0.00635" dist_x="0.135" dist_y="0.2" dist_z="0.25505" wr="0" wp="0" wy="0" density="650" />
+		<xacro:create_mesh name="BaseLV4" size_x="0.25" size_y="0.25" size_z="0.00635" dist_x="0.0008" dist_y="0.125" dist_z="0.7114" wr="0" wp="0" wy="0" density="650" />
+		<xacro:create_mesh name="Suporte" size_x="0.12607" size_y="0.12607" size_z="0.009" dist_x="-0.06117" dist_y="0.063035" dist_z="0.20605" wr="0" wp="0" wy="0" density="650" />
+		<xacro:create_mesh name="PlatMovelLV1" size_x="0.2054" size_y="0.19661" size_z="0.01" dist_x="-0.0215" dist_y="0.098305" dist_z="0.33745" wr="0" wp="0" wy="0" density="650" />
+		<xacro:create_mesh name="PlatMovelLV2" size_x="0.25" size_y="0.25" size_z="0.01" dist_x="0.0008" dist_y="0.125" dist_z="0.76745" wr="0" wp="0" wy="0" density="650" />
+		<xacro:create_cylinder name="C_LV1_1" radius="0.00635" height="0.0381" pos_x="0.14" pos_y="0.05443" pos_z="-0.02" wr="0" wp="0" wy="0" density="800" />
+		<xacro:create_cylinder name="C_LV1_2" radius="0.00635" height="0.0381" pos_x="0.14" pos_y="-0.05443" pos_z="-0.02" wr="0" wp="0" wy="0" density="800" />
+		<xacro:create_cylinder name="C_LV1_3" radius="0.00635" height="0.0381" pos_x="0.05" pos_y="0.1142" pos_z="-0.02" wr="0" wp="0" wy="0" density="800" />
+		<xacro:create_cylinder name="C_LV1_4" radius="0.00635" height="0.0381" pos_x="0.05" pos_y="-0.1142" pos_z="-0.02" wr="0" wp="0" wy="0" density="800" />
+		<xacro:create_cylinder name="C_LV1_5" radius="0.00635" height="0.0381" pos_x="-0.07" pos_y="0.1142" pos_z="-0.02" wr="0" wp="0" wy="0" density="800" />
+		<xacro:create_cylinder name="C_LV1_6" radius="0.00635" height="0.0381" pos_x="-0.07" pos_y="-0.1142" pos_z="-0.02" wr="0" wp="0" wy="0" density="800" />
+		<xacro:create_cylinder name="C_LV1_7" radius="0.00635" height="0.0381" pos_x="-0.19" pos_y="0.07843" pos_z="-0.02" wr="0" wp="0" wy="0" density="800" />
+		<xacro:create_cylinder name="C_LV1_8" radius="0.00635" height="0.0381" pos_x="-0.19" pos_y="-0.07843" pos_z="-0.02" wr="0" wp="0" wy="0" density="800" />
+		<xacro:create_cylinder name="C_LV1_9" radius="0.00635" height="0.0381" pos_x="-0.27" pos_y="0" pos_z="-0.02" wr="0" wp="0" wy="0" density="800" />
+		<xacro:create_cylinder name="C_LV2_1" radius="0.00635" height="0.226" pos_x="0.085" pos_y="0.115" pos_z="0.12205" wr="0" wp="0" wy="0" density="800" />
+		<xacro:create_cylinder name="C_LV2_2" radius="0.00635" height="0.226" pos_x="0.085" pos_y="-0.115" pos_z="0.12205" wr="0" wp="0" wy="0" density="800" />
+		<xacro:create_cylinder name="C_LV2_3" radius="0.00635" height="0.226" pos_x="-0.125" pos_y="0.115" pos_z="0.12205" wr="0" wp="0" wy="0" density="800" />
+		<xacro:create_cylinder name="C_LV2_4" radius="0.00635" height="0.226" pos_x="-0.125" pos_y="-0.115" pos_z="0.12205" wr="0" wp="0" wy="0" density="800" />
+		<xacro:create_cylinder name="C_LV2_5" radius="0.00635" height="0.226" pos_x="-0.2492" pos_y="0" pos_z="0.12205" wr="0" wp="0" wy="0" density="800" />
+		<xacro:create_cylinder name="C_SPT_1" radius="0.00635" height="0.05" pos_x="-0.07117" pos_y="0" pos_z="0.22005" wr="0" wp="0" wy="0" density="800" />
+		<xacro:create_cylinder name="C_SPT_2" radius="0.00635" height="0.05" pos_x="-0.125" pos_y="0.05303" pos_z="0.22005" wr="0" wp="0" wy="0" density="800" />
+		<xacro:create_cylinder name="C_SPT_3" radius="0.00635" height="0.05" pos_x="-0.125" pos_y="-0.05303" pos_z="0.22005" wr="0" wp="0" wy="0" density="800" />
+		<xacro:create_cylinder name="C_SPT_4" radius="0.00635" height="0.05" pos_x="-0.17723" pos_y="0" pos_z="0.22005" wr="0" wp="0" wy="0" density="800" />
+		<xacro:create_cylinder name="C_LV3_1" radius="0.00635" height="0.448" pos_x="-0.05349" pos_y="0.07071" pos_z="0.4754" wr="0" wp="0" wy="0" density="800" />
+		<xacro:create_cylinder name="C_LV3_2" radius="0.00635" height="0.448" pos_x="-0.05349" pos_y="-0.07071" pos_z="0.4754" wr="0" wp="0" wy="0" density="800" />
+		<xacro:create_cylinder name="C_LV3_3" radius="0.00635" height="0.448" pos_x="-0.19491" pos_y="0.07071" pos_z="0.4754" wr="0" wp="0" wy="0" density="800" />
+		<xacro:create_cylinder name="C_LV3_4" radius="0.00635" height="0.448" pos_x="-0.19491" pos_y="-0.07071" pos_z="0.4754" wr="0" wp="0" wy="0" density="800" />
+		<xacro:create_cylinder name="C_GUIA_1" radius="0.00635" height="0.5" pos_x="-0.04635" pos_y="0" pos_z="0.5014" wr="0" wp="0" wy="0" density="800" />
+		<xacro:create_cylinder name="C_GUIA_2" radius="0.00635" height="0.5" pos_x="-0.20135" pos_y="0" pos_z="0.5014" wr="0" wp="0" wy="0" density="800" />
+		<xacro:create_cylinder name="C_PLT_1" radius="0.00635" height="0.42" pos_x="-0.06632" pos_y="0.02252" pos_z="0.54745" wr="0" wp="0" wy="0" density="800" />
+		<xacro:create_cylinder name="C_PLT_2" radius="0.00635" height="0.42" pos_x="-0.1242" pos_y="0.0804" pos_z="0.54745" wr="0" wp="0" wy="0" density="800" />
+		<xacro:create_cylinder name="C_PLT_3" radius="0.00635" height="0.42" pos_x="-0.1242" pos_y="0.0804" pos_z="0.54745" wr="0" wp="0" wy="0" density="800" />
+		<xacro:create_cylinder name="C_PLT_4" radius="0.00635" height="0.42" pos_x="-0.18208" pos_y="-0.02252" pos_z="0.54745" wr="0" wp="0" wy="0" density="800" />
+		<xacro:create_cylinder name="C_BODY" radius="0.0125" height="0.506" pos_x="-0.1242" pos_y="0" pos_z="0.49055" wr="0" wp="0" wy="0" density="800" />
 		<!--
 		<xacro:create_cylinder name="chassis" mass="${body_mass}" radius="${body_radius}" length="${body_length}"
@@ -99,5 +99,5 @@
 		<link name="zed_camera_center">
 			<visual>
-				<origin xyz="0 0 0" rpy="0 0 0"/>
+				<origin xyz="-0.05 0 0" rpy="0 0 0"/>
 				<geometry>
 					<mesh filename="package://zed_wrapper/urdf/models/ZED.stl" />
